Commit message: Add gimbal gazebo plugin, applying in task1 to stabilize the camera.

File: jsk_mbzirc_tasks/urdf/quadrotor_with_hokyo30lx_and_downward_cam.urdf.xacro (robot description, xacro)
@@ -8,13 +8,19 @@
     <xacro:property name="M_PI" value="3.1415926535897931" />
     <!-- Custom sensors settings -->
-    <!-- Hokuyo UTM-30LX mounted upside down below the quadrotor body -->
+    <!-- Hokuyo UTM-30LX mounted on the quadrotor body -->
     <xacro:include filename="$(find hector_sensors_description)/urdf/hokuyo_utm30lx.urdf.xacro" />
     <xacro:hokuyo_utm30lx name="laser0" parent="base_link" ros_topic="scan" update_rate="40" ray_count="1081" min_angle="-135" max_angle="135">
-      <origin xyz="0.0 0.0 -0.097" rpy="${M_PI} 0 0"/>
+      <origin xyz="0.0 0.0 0.097" rpy="0 0 0"/>
     </xacro:hokuyo_utm30lx>
-    <!-- Downward facing camera -->
+    <!-- Downward facing camera with Gimbal -->
+    <!-- Gimabal -->
+    <xacro:include filename="$(find jsk_mbzirc_tasks)/urdf/gimbal/gimbal.xacro" />
+    <xacro:gimbal name="gimbal" parent="base_link" topside="false" width="0.015" motor_height="0.015" x="0.04" y="0.03" z="0.06" imu_topic_name="/raw_imu">
+      <origin xyz="-0.05 0.0 -0.04" rpy="0 0 0"/>
+    </xacro:gimbal>
+    <!-- Camera -->
     <xacro:include filename="$(find hector_sensors_description)/urdf/generic_camera.urdf.xacro" />
-    <xacro:generic_camera name="downward_cam" parent="base_link" ros_topic="camera/image" cam_info_topic="camera/camera_info" update_rate="20" res_x="640" res_y="480" image_format="L8" hfov="100">
-      <origin xyz="0.4 0.0 -0.0" rpy="0 ${M_PI/2} 0"/>
+    <xacro:generic_camera name="downward_cam" parent="gimbal_stabilized_link" ros_topic="camera/image" cam_info_topic="camera/camera_info" update_rate="20" res_x="640" res_y="480" image_format="L8" hfov="160">
+      <origin xyz="0.0 0.0 -0.03" rpy="0 ${M_PI/2} 0"/>
     </xacro:generic_camera>
 </robot>
